File: VGA.kicad_pcb (KiCad board)
At the start: 4 copper layers, 269.5 x 146.7 mm, 14 parts, among them U15 4464, U16 4464, U21 4464, U22 4464, U28 4464, U29 4464, U8 4464, U9 4464

Commit message: Add files via upload
Connections:
- net /A4_3 renamed /A4_2
- net /A5_3 renamed /A5_2
- RN5 pad 3: unconnected-(RN5-R2-Pad3) -> /RAS3
- U15 pad 16: unconnected-(U15-~{CAS}-Pad16) -> /CAS3
- U15 pad 18: +5V -> GND
- U15 pad 5: unconnected-(U15-~{RAS}-Pad5) -> /RAS3
- U15 pad 6: /A6_3 -> /A6_2
- U15 pad 9: GND -> +5V
- U16 pad 18: +5V -> GND
- U16 pad 6: /A6_ -> /A6
- U16 pad 7: /A5_ -> /A5
- U16 pad 8: /A4_ -> /A4
- U16 pad 9: GND -> +5V
- U21 pad 16: unconnected-(U21-~{CAS}-Pad16) -> /CAS3
- U21 pad 18: +5V -> GND
- U21 pad 5: unconnected-(U21-~{RAS}-Pad5) -> /RAS3
- U21 pad 6: /A6_3 -> /A6_2
- U21 pad 9: GND -> +5V
- U22 pad 18: +5V -> GND
- U22 pad 9: GND -> +5V
- U28 pad 16: unconnected-(U28-~{CAS}-Pad16) -> /CAS2
- U28 pad 18: +5V -> GND
- U28 pad 5: unconnected-(U28-~{RAS}-Pad5) -> /RAS2
- U28 pad 6: /A6_3 -> /A6_2
- U28 pad 9: GND -> +5V
- U29 pad 18: +5V -> GND
- U29 pad 9: GND -> +5V
- U8 pad 16: unconnected-(U8-~{CAS}-Pad16) -> /CAS2
- U8 pad 18: +5V -> GND
- U8 pad 5: unconnected-(U8-~{RAS}-Pad5) -> /RAS2
- U8 pad 6: /A6_3 -> /A6_2
- U8 pad 9: GND -> +5V
- U9 pad 18: +5V -> GND
- U9 pad 6: /A6_ -> /A6
- U9 pad 7: /A5_ -> /A5
- U9 pad 8: /A4_ -> /A4
- U9 pad 9: GND -> +5V
Routing:
- net (no net): track 1595.6 -> 2054.2 mm, vias 57 -> 56
- net /A6_3: track 84.4 -> 0.00 mm
- net /A6_2: track 0.00 -> 84.4 mm
- net /A5_: track 74.5 -> 0.00 mm
- net /RAS3: track 0.00 -> 74.2 mm, vias 0 -> 1
- net unconnected-(RN5-R2-Pad3): track 46.5 -> 0.00 mm, vias 1 -> 0
- net /CAS2: track 0.00 -> 32.3 mm
- net /A4: track 18.2 -> 33.8 mm
- net /RAS2: track 0.00 -> 13.8 mm, vias 0 -> 1
- net /A5: track 20.6 -> 33.8 mm
- net /A6: track 57.4 -> 70.4 mm
- net /A6_: track 11.3 -> 0.00 mm
- net /A4_: track 11.3 -> 0.00 mm
- net /CAS3: track 0.00 -> 11.2 mm
- net unconnected-(U8-~{CAS}-Pad16): track 6.09 -> 0.00 mm
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