File: VGA.kicad_sch (KiCad schematic)
At the start: 14 parts, among them U15 4464, U16 4464, U21 4464, U22 4464, U28 4464, U29 4464, U8 4464, U9 4464

Commit message: Add files via upload
Connections:
- net A4_ is gone; now on net A4: U16.8 (A4), U9.8 (A4)
- net A5_ is gone; now on net A5: U16.7 (A5), U9.7 (A5)
- net A6_ is gone; now on net A6: U16.6 (A6), U9.6 (A6)
- net +5V: now also U15.9 (VCC), U16.9 (VCC), U21.9 (VCC), U22.9 (VCC), U28.9 (VCC), U29.9 (VCC), U8.9 (VCC), U9.9 (VCC); no longer U15.18 (VSS), U16.18 (VSS), U21.18 (VSS), U22.18 (VSS), U28.18 (VSS), U29.18 (VSS), U8.18 (VSS), U9.18 (VSS)
- net A6_3: no longer U15.6 (A6), U21.6 (A6), U28.6 (A6), U8.6 (A6)
- net GND: now also U15.18 (VSS), U16.18 (VSS), U21.18 (VSS), U22.18 (VSS), U28.18 (VSS), U29.18 (VSS), U8.18 (VSS), U9.18 (VSS); no longer U15.9 (VCC), U16.9 (VCC), U21.9 (VCC), U22.9 (VCC), U28.9 (VCC), U29.9 (VCC), U8.9 (VCC), U9.9 (VCC)
- net CAS2: now reaches U8.16 (~{CAS})
- net CAS2: now also U28.16 (~{CAS})
- net RAS2: now reaches U8.5 (~{RAS})
- net RAS2: now also U28.5 (~{RAS})
- net RAS3: now reaches RN5.3 (R2)
- net RAS3: now also U15.5 (~{RAS}), U21.5 (~{RAS})
- net CAS3: now reaches U15.16 (~{CAS})
- net CAS3: now also U21.16 (~{CAS})
- net A4_3 renamed A4_2
- net A5_3 renamed A5_2
- new net A6_2: U15.6 (A6), U21.6 (A6), U28.6 (A6), U8.6 (A6)
Other:
- moved on the sheet: RN10, RN11, RN5, RN6, RN7
